File: Page2(output).kicad_sch (KiCad schematic)
At the start: 84 parts, among them K1 SRD-12VDC-SL-C, K2 SRD-12VDC-SL-C, K3 SRD-12VDC-SL-C, K4 SRD-12VDC-SL-C, K5 SRD-12VDC-SL-C, K6 SRD-12VDC-SL-C, P1 zx-xh2.54, Q1 SS8050, Q2 SS8050, U10 LTV-358T, U11 LTV-358T, U12 LTV-358T, U13 LTV-358T, U14 LTV-358T, U15 PCF8574P, U16 PCF8574P, U17 74HCT14D_653, U18 ULN2003A, U19 74HCT14D_653, U20 ULN2003A, U21 74HCT14D_653, U22 ULN2003A, U23 74HCT14D_653, U24 ULN2003A, U9 LTV-358T

Commit message: :Zap:making chngs to powerinput, and relay output
Parts:
- removed C17, C19, C20, C21, C26, C29, C32: 100nF, Capacitor_Tantalum_SMD:CP_EIA-3216-18_Kemet-A, symbol Device:C
- removed K1, K2, K3, K4, K5, K6: SRD-12VDC-SL-C, SRD-12VDC-SL-C:RELAY_SRD-12VDC-SL-C, symbol SRD-12VDC-SL-C:SRD-12VDC-SL-C
- removed P1: zx-xh2.54, Inductor_SMD:L_Sunlord_MWSA0605S, symbol Connector_Generic:Conn_01x04
- removed Q1, Q2: SS8050, Package_TO_SOT_SMD:SOT-23, symbol Transistor_BJT:SS8050
- removed R30, R31: 10k, Resistor_SMD:R_0805_2012Metric, symbol Device:R
- removed R32, R33: 100R, Resistor_SMD:R_1218_3246Metric, symbol Device:R
- removed R34, R35: 12k, Resistor_SMD:R_0805_2012Metric, symbol Device:R
- removed R44, R45, R46, R47, R48, R49: 100K, Resistor_SMD:R_1218_3246Metric, symbol Device:R
- removed R51, R52, R53: 10K, Resistor_THT:R_Axial_DIN0614_L14.3mm_D5.7mm_P5.08mm_Vertical, symbol Device:R
- removed R60, R61, R62, R63, R64, R65: 4.7K, Resistor_SMD:R_1206_3216Metric, symbol Device:R
- removed RN1, RN2: R_Network04, Resistor_THT:R_Array_SIP5, symbol Device:R_Network04
- removed S1, S2: B3U-1000P, B3U-1000P:SW_B3U-1000P, symbol B3U-1000P:B3U-1000P
- removed U16: PCF8574P, Package_DIP:DIP-16_W7.62mm, symbol Interface_Expansion:PCF8574P
- removed U17, U19, U21, U23: 74HCT14D_653, 74HCT14D_653:SOIC127P600X175-14N, symbol 74hct14d_653:74HCT14D_653
- added U7: PC817, Package_DIP:DIP-4_W7.62mm, symbol Isolator:PC817
Connections:
- net +12VIN: no longer C22.1, C23.1, D11.2 (A), D12.2 (A), D13.2 (A), D14.2 (A), D15.2 (A), D16.2 (A), U10.1, U11.1, U12.1, U13.1, U14.1, U18.9 (COM), U9.1
- new net +24VIN: D11.2 (A), D12.2 (A), D13.2 (A), D14.2 (A), D15.2 (A), D16.2 (A), U10.1, U11.1, U12.1, U13.1, U14.1, U9.1
- new net 24VIN: C22.1, C23.1, U18.9 (COM)
- no-connect marks 12 -> 7
Other:
- note removed: "PROG"

Commit message: :rocket:Have added Ethernet BUFFER and CONNECTED TO STM
Parts:
- added J4: Screw_Terminal_01x06, symbol Connector:Screw_Terminal_01x06
- added R51, R52, R53, R60, R61, R62, R63, R64, R65, R66, R67, R68, R76, R77, R78: 4.7K, Resistor_THT:R_Axial_DIN0614_L14.3mm_D5.7mm_P5.08mm_Vertical, symbol Device:R
- added U16, U17, U19, U21, U23, U25, U26, U27, U28, U29, U30, U31, U32, U33: PC817, Package_DIP:DIP-4_W7.62mm, symbol Isolator:PC817
Connections:
- net +12VIN: no longer C27.1, C30.1, C33.1, U20.9 (COM), U22.9 (COM), U24.9 (COM)
- net +24VIN: now also C27.1, C30.1, C33.1, U20.9 (COM), U22.9 (COM), U24.9 (COM)
- net GND: now also U7.3, U16.3, U17.3, U19.3, U21.3, U23.3, U25.3, U26.3, U27.3, U28.3, U29.3, U30.3, U31.3, U32.3, U33.3
- net OUT10: now also R63.1
- net OUT11: now also R62.1
- net OUT12: now also R61.1
- net OUT21: now also R78.1
- net OUT22: now also R77.1
- net OUT23: now also R76.1
- net OUT24: now also R68.1
- net OUT3: now also R60.1
- net OUT4: now also R53.1
- net OUT5: now also R51.1
- net OUT6: now also R52.1, R67.1
- net OUT8: now also R65.1
- net OUT9: now also R64.1, R66.1
- net +24V: now reaches U7.1
- net +24V: now also U16.1, U17.1, U19.1, U21.1, U23.1, U25.1, U26.1, U27.1, U28.1, U29.1, U30.1, U31.1, U32.1, U33.1
- net at U7.2: now also R51.2
- new net: R65.2, U27.2
- new net: R67.2, U29.2
- new net: R68.2, U30.2
- new net: R64.2, U26.2
- new net: R61.2, U21.2
- new net: R62.2, U23.2
- new net: R63.2, U25.2
- new net: R77.2, U32.2
- new net: R78.2, U33.2
- new net: R53.2, U17.2
- new net: R60.2, U19.2
- new net: R76.2, U31.2
- new net: R66.2, U28.2
- new net: R52.2, U16.2

Commit message: :wrench: Connecting opto to the relay
Connections:
- net PE8: now reaches U27.4
- net PC7: now reaches U29.4
- net PE5: now reaches U23.4
- net PE6: now reaches U25.4
- net PC10: now reaches U32.4
- net PC11: now reaches U33.4
- net PE2: now reaches U17.4
- net PC9: now reaches U31.4
- net PE4: now reaches U21.4
- net PE7: now reaches U26.4
- net PE0: now reaches U16.4
- net PE3: now reaches U19.4
- net PC8: now reaches U30.4
- net PC6: now reaches U28.4
- net PE1: now reaches U7.4

Commit message: :tada: Completing minor touches
Parts:
- removed R50: 10K, Resistor_THT:R_Axial_DIN0614_L14.3mm_D5.7mm_P5.08mm_Vertical, symbol Device:R
- removed U15: PCF8574P, Package_DIP:DIP-16_W7.62mm, symbol Interface_Expansion:PCF8574P
Connections:
- net INPUT D1: now also J4.6 (Pin_6)
- net INPUT D2: now also J4.5 (Pin_5)
- net INPUT D3: now also J4.4 (Pin_4)
- net INPUT D4: now also J4.3 (Pin_3)
- net INPUT D5: now also J4.2 (Pin_2), R42.2
- net INPUT D6: now also J4.1 (Pin_1), R43.2
- no-connect marks 7 -> 4
Other:
- moved on the sheet: D11, D12, D13, D14, D15, D16, J4, R38, R39, R40, R41, R42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
